Commit message: wip

File: pybullet-helpers/src/pybullet_helpers/assets/urdf/tidybot/tidybot_base.urdf (robot description, URDF)
Before this commit: robot tidybot_base, 1 links, 0 joints
Links:
- added link base_root
Joints:
- added joint base_root_to_base_link: type fixed, parent base_root, child base_link, origin xyz=0 0 0 rpy=0 0 0

Commit message: wip

File: pybullet-helpers/src/pybullet_helpers/assets/urdf/tidybot/tidybot_base.urdf (robot description, URDF)
Before this commit: robot tidybot_base, 2 links, 1 joints
Links:
- link base_link: mass 60 -> 0; geometry collision box size=0.548 0.508 0.29; collision mesh filename=meshes/arm_plate.stl

Commit message: wip

File: pybullet-helpers/src/pybullet_helpers/assets/urdf/tidybot/tidybot_base.urdf (robot description, URDF)
Before this commit: robot tidybot_base, 2 links, 1 joints
Links:
- link base_link: geometry collision box size=0.548 0.508 0.29; visual mesh filename=meshes/arm_plate.stl

Commit message: wip

File: pybullet-helpers/src/pybullet_helpers/assets/urdf/tidybot/tidybot_base.urdf (robot description, URDF)
Before this commit: robot tidybot_base, 2 links, 1 joints
Links:
- link base_link: geometry collision box size=0.548 0.508 0.365; visual mesh filename=meshes/arm_plate.stl
