Commit message: wip

File: pybullet-helpers/src/pybullet_helpers/assets/urdf/kortex_description/gen3_7dof.urdf (robot description, URDF)
Before this commit: robot gen3_robotiq_2f_85, 24 links, 23 joints
Links:
- link robotiq_arg2f_base_link: geometry collision mesh filename=package://kortex_description/grippers/robotiq_2f_85/meshes/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 scale=0.001 0.001 0.001; visual mesh filename=package://kortex_description/grippers/robotiq_2f_85/meshes/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 scale=0.001 0.001 0.001

Commit message: wip

File: pybullet-helpers/src/pybullet_helpers/assets/urdf/kortex_description/gen3_7dof.urdf (robot description, URDF)
Before this commit: robot gen3_robotiq_2f_85, 24 links, 23 joints
Links:
- link robotiq_arg2f_base_link: geometry collision mesh filename=package://kortex_description/grippers/robotiq_2f_85/meshes/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; visual mesh filename=package://kortex_description/grippers/robotiq_2f_85/meshes/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 scale=0.001 0.001 0.001

Commit message: add wrist camera to kinova gen3 collision geometry (#322)

File: pybullet-helpers/src/pybullet_helpers/assets/urdf/kortex_description/gen3_7dof.urdf (robot description, URDF)
Before this commit: robot gen3_robotiq_2f_85, 24 links, 23 joints
Links:
- link robotiq_arg2f_base_link: geometry collision box size=0.025 0.09 0.035; collision mesh filename=package://kortex_description/grippers/robotiq_2f_85/meshes/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
