Commit message: set Vega gripper tool frame to the fingertip TCP
L_ee/R_ee were zero-offset frames at the wrist flange, so an IK/grasp target at an
object placed the long fingers ~0.25 m beyond it (into the table for a top-down
grasp). Move them 0.23 m down the gripper approach axis to the fingertip pads, so a
zero-offset grasp targets the actual grasp point -- matching the convention the
Panda and Kinova tool frames already follow.

Co-Authored-By: Claude Opus 4.8 (1M context) <noreply@anthropic.com>

File: prpl-kinematics/src/prpl_kinematics/assets/urdf/vega/vega_1u_gripper.urdf (robot description, URDF)
Before this commit: robot vega_1u_gripper, 34 links, 33 joints
Joints:
- joint L_ee_j0: origin xyz=0 0 0 rpy=0 0 -1.57079 -> xyz=0 0 0.23 rpy=0 0 -1.57079
- joint R_ee_j0: origin xyz=0 0 0 rpy=0 0 1.57079 -> xyz=0 0 0.2 rpy=0 0 1.57079

Commit message: prpl-kinematics: sync the Vega gripper model to the Dexgripper S (#532)
The bundled vega_1u_gripper.urdf modeled the Dexgripper D, one generation
behind the Dexgripper S hardware being mounted on the lab's Vega 1U. Sync the
URDF and gripper meshes to dexmate_urdf 0.8.4, which models the S: new gripper
meshes (fingers ~2.3x narrower), a remounted gripper base (+4.5 mm along the
wrist, -90 degree yaw with correspondingly rotated finger axes), updated
gripper and head_l2 inertials, and the same 0-0.7854 rad finger limits as
before. The two prpl modifications to the upstream file are re-applied and now
documented in make_vega: the L_ee/R_ee fingertip tool-frame offsets, and the
exclusion of the S's visual-only wrist-camera links (the lab unit has no wrist
camera). The stale dexd meshes are removed.

Verified against the pre-sync model: the L_ee/R_ee home poses are unchanged;
the finger closing axis in the ee frame is still +/-x (the mount yaw and the
new finger axes cancel); the finger hinges move ~1.5 mm in y and ~5 mm in z;
discover_allowed_pairs at home returns the identical 29-pair set; the full CI
suite passes (mypy, pylint, 92 tests).

Co-Authored-By: Claude Fable 5 <noreply@anthropic.com>

File: prpl-kinematics/src/prpl_kinematics/assets/urdf/vega/vega_1u_gripper.urdf (robot description, URDF)
Before this commit: robot vega_1u_gripper, 34 links, 33 joints
Links:
- link L_gripper_base: mass 0.39258 -> 0.217869646528476; geometry collision mesh filename=../../hands/dexs_gripper/meshes/collision/gripper_base.obj; visual mesh filename=../../hands/dexs_gripper/meshes/visual/gripper_base.glb
- link L_gripper_l1: mass 0.09974 -> 0.0417789910080777; geometry collision mesh filename=../../hands/dexs_gripper/meshes/collision/gripper_l1.obj; visual mesh filename=../../hands/dexs_gripper/meshes/visual/gripper_l1.glb
- link L_gripper_l2: mass 0.09973 -> 0.0417790873345589; geometry collision mesh filename=../../hands/dexs_gripper/meshes/collision/gripper_l2.obj; visual mesh filename=../../hands/dexs_gripper/meshes/visual/gripper_l2.glb
- link R_gripper_base: mass 0.39258 -> 0.217869646528476; geometry collision mesh filename=../../hands/dexs_gripper/meshes/collision/gripper_base.obj; visual mesh filename=../../hands/dexs_gripper/meshes/visual/gripper_base.glb
- link R_gripper_l1: mass 0.09974 -> 0.0417789910080777; geometry collision mesh filename=../../hands/dexs_gripper/meshes/collision/gripper_l1.obj; visual mesh filename=../../hands/dexs_gripper/meshes/visual/gripper_l1.glb
- link R_gripper_l2: mass 0.09973 -> 0.0417790873345589; geometry collision mesh filename=../../hands/dexs_gripper/meshes/collision/gripper_l2.obj; visual mesh filename=../../hands/dexs_gripper/meshes/visual/gripper_l2.glb
Joints:
- joint L_gripper_j1: axis -1 0 0 -> 0 -1 0; origin xyz=4.92002E-18 0.0258 0.02875 rpy=0 0 0 -> xyz=-0.025807 -0.0015 0.02935 rpy=0 0 0
- joint L_gripper_j2: axis 1 0 0 -> 0 1 0; origin xyz=-1.39916E-18 -0.0258 0.02875 rpy=0 0 0 -> xyz=0.025793 -0.0015 0.02935 rpy=0 0 0
- joint L_hand_mount: origin xyz=0.0 0 0.078 rpy=0 0 0 -> xyz=0.0 0 0.0825 rpy=0 0 -1.5708
- joint R_gripper_j1: axis -1 0 0 -> 0 -1 0; origin xyz=4.92002E-18 0.0258 0.02875 rpy=0 0 0 -> xyz=-0.025807 -0.0015 0.02935 rpy=0 0 0
- joint R_gripper_j2: axis 1 0 0 -> 0 1 0; origin xyz=-1.39916E-18 -0.0258 0.02875 rpy=0 0 0 -> xyz=0.025793 -0.0015 0.02935 rpy=0 0 0
- joint R_hand_mount: origin xyz=0 0 0.078 rpy=0 0 0 -> xyz=0 0 0.0825 rpy=0 0 -1.5708
